File: PANNEL_Final.brd (EAGLE design)
At the start: 85 x 246 mm, 152 parts, among them IC1 25LC1024-I/P, IC2 25LC1024-I/P, IC3 FGPMMOPA6H, IC4 FXAS21000, IC5 ADXL343BCCZ, IC6 MPL3115A2LGA, Q1 FQP7P06, Q2 FQP7P06, Q3 12MHz, Q4 MCP9700A-E/TO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

Commit message: SPELLING
Parts:
- added JP4: (no value), jumper:JP1
Connections:
- new net N$95: JP4.1, U3.28
- net GND: now also JP4.2
Routing:
- net N$95: track 0.00 -> 5.55 mm
Other:
- board text added: "BALANCED"
- board text added: "CU IN SPACE 2018"
- board text added: "PROPERTERY OF: CARLETON UNIVERSITY IN SPACE"
- board text added: "UNBALANCED"
- board text removed: "BALENCED"
- board text removed: "UNBALENCED"
Changed lines of the file:
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@@
 <text x="6.2738" y="176.3688" size="1.27" layer="125" ratio="10">JP2</text>
 <text x="31.8262" y="203.1912" size="1.27" layer="125" ratio="10" rot="R180">JP3</text>
-<text x="49.7078" y="196.13" size="2.0828" layer="125" ratio="10" rot="SR0">LM3950</text>
+<text x="48.9578" y="188.13" size="2.0828" layer="125" ratio="10" rot="SR0">LM3950</text>
 <text x="35.56" y="178.35" size="1.27" layer="125" rot="R90">XB1</text>
 <text x="42.164" y="194.606" size="1.27" layer="125" ratio="10" rot="R270">C1</text>
@@
 <text x="6.2738" y="176.3688" size="1.27" layer="125" ratio="10">JP2</text>
 <text x="31.8262" y="203.1912" size="1.27" layer="125" ratio="10" rot="R180">JP3</text>
-<text x="49.7078" y="196.13" size="2.0828" layer="125" ratio="10" rot="SR0">LM3950</text>
+<text x="48.9578" y="188.13" size="2.0828" layer="125" ratio="10" rot="SR0">LM3950</text>
 <text x="35.56" y="178.35" size="1.27" layer="125" rot="R90">XB1</text>
 <rectangle x1="27.2" y1="232.65" x2="42.8" y2="235.35" layer="1"/>
@@
 <rectangle x1="66.55" y1="229.25" x2="71.75" y2="245.8" layer="29"/>
 <rectangle x1="66.55" y1="211.25" x2="71.75" y2="227.8" layer="29"/>
-<text x="3.45" y="240.6" size="1.778" layer="21">BALENCED</text>
-<text x="34.45" y="240.5" size="1.778" layer="21">UNBALENCED</text>
+<text x="38.2" y="239.85" size="1.778" layer="21">BALANCED</text>
+<text x="1.45" y="239.75" size="1.778" layer="21">UNBALANCED</text>
 <rectangle x1="1.05" y1="228" x2="6.6" y2="229" layer="1"/>
 <rectangle x1="6.6" y1="228" x2="13.95" y2="229" layer="1"/>
@@
 <vertex x="73.5" y="229"/>
 </polygon>
+<text x="36" y="197.25" size="1.778" layer="21">PROPERTERY OF:
+CARLETON UNIVERSITY IN SPACE</text>
+<text x="32.25" y="215.5" size="1.778" layer="21">CU IN SPACE 2018</text>
 </plain>
 <attributes>
@@
 <element name="LM3950" library="CU-InSpace_Ground" package="TO254P470X1016X2222-3P" value="LM3940IT-3.3" x="52.07" y="192.32" smashed="yes" rot="R180">
 <attribute name="MPN" value="LM3940IT-3.3" x="52.07" y="192.32" size="1.778" layer="27" rot="R180" display="off"/>
-<attribute name="NAME" x="49.7078" y="196.13" size="2.0828" layer="25" ratio="10" rot="SR0"/>
+<attribute name="NAME" x="48.9578" y="188.13" size="2.0828" layer="25" ratio="10" rot="SR0"/>
 <attribute name="OC_FARNELL" value="9494553" x="52.07" y="192.32" size="1.778" layer="27" rot="R180" display="off"/>
 <attribute name="OC_NEWARK" value="41K5126" x="52.07" y="192.32" size="1.778" layer="27" rot="R180" display="off"/>
 <attribute name="PACKAGE" value="TO-220" x="52.07" y="192.32" size="1.778" layer="27" rot="R180" display="off"/>
 <attribute name="SUPPLIER" value="NATIONAL SEMICONDUCTOR" x="52.07" y="192.32" size="1.778" layer="27" rot="R180" display="off"/>
-<attribute name="VALUE" x="60.2234" y="197.8572" size="2.0828" layer="27" ratio="10" rot="SR180"/>
 </element>
 <element name="JP1" library="pinhead" library_urn="urn:adsk.eagle:library:325" package="1X04" package3d_urn="urn:adsk.eagle:package:22407/2" value="" x="82.15" y="191.05" smashed="yes" rot="R90">
@@
 <attribute name="VALUE" x="43.603" y="220.079" size="1.27" layer="27"/>
 </element>
+<element name="JP4" library="jumper" library_urn="urn:adsk.eagle:library:252" package="JP1" package3d_urn="urn:adsk.eagle:package:15455/1" value="" x="37.75" y="10.75" rot="R90"/>
 </elements>
 <signals>
@@
 <wire x1="20.7" y1="18.1938" x2="20.7" y2="16" width="0.254" layer="1"/>
 <wire x1="20.7" y1="16" x2="22.05" y2="16.35" width="0.254" layer="1"/>
+<contactref element="JP4" pad="2"/>
 </signal>
 <signal name="N$73">
@@
 <contactref element="T5" pad="1"/>
 </signal>
+<signal name="N$95">
+<contactref element="U3" pad="28"/>
+<contactref element="JP4" pad="1"/>
+<wire x1="42.71" y1="14.77" x2="42.71" y2="14.44" width="0.254" layer="1"/>
+<wire x1="42.71" y1="14.44" x2="39.02" y2="10.75" width="0.254" layer="1"/>
+</signal>
 </signals>
 <errors>
@@
 </drawing>
 <compatibility>
+<note version="6.3" minversion="6.2.2" severity="warning">
+Since Version 6.2.2 text objects can contain more than one line,
+which will not be processed correctly with this version.
+</note>
 <note version="8.2" severity="warning">
 Since Version 8.2, EAGLE supports online libraries. The ids
