File: main.sch (EAGLE design)
At the start: 128 parts, among them IC1 FXAS21000, IC2 ADXL343BCCZ, IC3 MPL3115A2LGA, IC4 FGPMMOPA6H, IC5 25LC1024-I/P, IC6 25LC1024-I/P, Q1 MCP9700A-E/TO, Q2 MCP9700A-E/TO, Q3 12MHz, Q4 FQP7P06, U1 ATMEGA1284P-PU, U2 LT3570EFEPBF, U3 TL431BQLP, X1 132134RP

Commit message: Update
Parts:
- removed ARMED: RED, led:LED5MM
- removed DC1: PJ-102BH, Power:PJ-102BH
- removed PAD4: (no value), Power:CRIMP
- removed SJ6: (no value), jumper:SJ
- removed U$8: BAT+, Power:TEST
- added ARMED1, ARMED2: RED, led:LED5MM
- added C34: 10µF, rcl:CPOL-USE2-5
- added C35, C36, C37: 0.1µF, rcl:C-EU025-025X050
- added Q5: MCP9700A-E/TO, CU in Space:MCP9700A-E/TO
- added R45, R48: (no value), rcl:R-US_0207/5V
- added R46, R47: 47kΩ, rcl:R-US_0207/5V
- added R49, R50: 2k2Ω, rcl:R-US_0207/5V
- added SJ200: (no value), jumper:SJ
- added T4: (no value), Power:-NPN_DARL-
- C1, C14, C2: value 0.1µF -> 22µF; device rcl:C-EU025-025X050 -> Power:UST1V220MDD
- C11, C4: value 0.1µF -> 338TTA035M; device rcl:C-EU025-025X050 -> Power:338TTA035M
- C12: value 0.1µF -> SNUB
- C13, C3, C7: value 0.1µF -> 10 uF; device rcl:C-EU025-025X050 -> Power:K102K15X7RF5TL2
- C15: value 2.2µF -> 338TTA035M; device rcl:C-EU025-025X050 -> Power:338TTA035M
- C16: value 27pF -> 1µF
- C17: value 27pF -> 0.1µF
- C18: value 0.1µF -> 47pF
- C19: value 47pF -> 0.1µF
- C20: value 1µF -> 27pF
- C21: value 0.1µF -> 27pF
- C22, C23: value 338TTA035M -> 0.1µF; device Power:338TTA035M -> rcl:C-EU025-025X050
- C24: value 338TTA035M -> 2.2µF; device Power:338TTA035M -> rcl:C-EU025-025X050
- C25, C26, C27: value 22µF -> 0.1µF; device Power:UST1V220MDD -> rcl:C-EU025-025X050
- C29, C31: value 10nF -> 0.1µF; device Power:K103K15X7RF5TL2 -> rcl:C-EU025-025X050
- C30: value 1nF -> 10µF; device Power:K102K15X7RF5TL2 -> rcl:CPOL-USE2-5
- C32: value 1nF -> 0.1µF; device Power:K102K15X7RF5TL2 -> rcl:C-EU025-025X050
- C5, C9: value 0.1µF -> 1nF; device rcl:C-EU025-025X050 -> Power:K102K15X7RF5TL2
- C6, C8: value 10µF -> 10nF; device rcl:CPOL-USE2-5 -> Power:K103K15X7RF5TL2
- IC1: value FXAS21000 -> 25LC1024-I/P; device Freescale_Sensors_v2:FXAS21000 -> microchip:25LC080P
- IC2: value ADXL343BCCZ -> 25LC1024-I/P; device CU in Space:ADXL343BCCZ -> microchip:25LC080P
- IC3: value MPL3115A2LGA -> FGPMMOPA6H; device microbuilder:MPL3115A2LGA -> microbuilder:GPS_FGPMMOPA6H
- IC4: value FGPMMOPA6H -> FXAS21000; device microbuilder:GPS_FGPMMOPA6H -> Freescale_Sensors_v2:FXAS21000
- IC5: value 25LC1024-I/P -> ADXL343BCCZ; device microchip:25LC080P -> CU in Space:ADXL343BCCZ
- IC6: value 25LC1024-I/P -> MPL3115A2LGA; device microchip:25LC080P -> microbuilder:MPL3115A2LGA
- L1: value 10µH -> 18µH; device rcl:L-US0207/5V -> Power:RLB0914-180KL
- L3: value 4.7µH -> 10µH; device Power:B78108E1472K000 -> rcl:L-US0207/5V
- Q1, Q2: value MCP9700A-E/TO -> FQP7P06; device CU in Space:MCP9700A-E/TO -> Power:FQP7P06
- Q4: value FQP7P06 -> MCP9700A-E/TO; device Power:FQP7P06 -> CU in Space:MCP9700A-E/TO
- R1: value 47kΩ -> 3.65 kΩ
- R10: value 1KΩ -> 51.1 kΩ
- R11: value 1MΩ -> BOOSTR
- R12: value 1M -> 1.2 k; device Power:MFR-25FBF52-3K65 -> rcl:R-US_0207/5V
- R13: value 3.6k -> SNUB; device Power:MFR-25FBF52-3K65 -> rcl:R-US_0207/5V
- R14: value 1MΩ -> 3.6k
- R15: value 750 -> 1.2 k; device Power:MFR-25FBF52-3K65 -> rcl:R-US_0207/5V
- R16: value 750 -> 3.6 k; device Power:MFR-25FBF52-3K65 -> rcl:R-US_0207/5V
- R17, R19: value 750 -> 1 M; device Power:MFR-25FBF52-3K65 -> rcl:R-US_0207/5V
- R18: value 750 -> 3.6 K; device Power:MFR-25FBF52-3K65 -> rcl:R-US_0207/5V
- R2: value (none) -> 1 MΩ; device Power:MFR-25FBF52-3K65 -> rcl:R-US_0207/5V
- R20: value 750 -> 1.4 k; device Power:MFR-25FBF52-3K65 -> rcl:R-US_0207/5V
- R21, R22, R23, R24, R25, R26, R27, R28: value 750 -> (none); device Power:MFR-25FBF52-3K65 -> rcl:R-US_0207/5V
- R29: value 750 -> 2M Ω; device Power:MFR-25FBF52-3K65 -> rcl:R-US_0207/5V
- R3: value 2k2Ω -> 1 MΩ
- R30: value ~1.4k -> 1MΩ; device Power:MFR-25FBF52-3K65 -> rcl:R-US_0207/5V
- R31, R34, R40: value 51.1kΩ -> (none); device Power:MFR-25FBF52-51K1 -> rcl:R-US_0207/5V
- R32: value 24.9kΩ -> 1.2 k; device Power:MFR-25FBF52-24K9 -> rcl:R-US_0207/5V
- R33: value 3.65kΩ -> 1.2k; device Power:MFR-25FBF52-3K65 -> rcl:R-US_0207/5V
- R35: value 17.4kΩ -> (none); device Power:MFR-25FBF52-17K4 -> rcl:R-US_0207/5V
- R36: value 8.06kΩ -> (none); device Power:MFR-25FBF52-8K06 -> rcl:R-US_0207/5V
- R37: value 3.65kΩ -> 1MΩ; device Power:MFR-25FBF52-3K65 -> rcl:R-US_0207/5V
- R38: value 24.9kΩ -> (none); device Power:MFR-25FBF52-24K9 -> rcl:R-US_0207/5V
- R39: value 1M -> (none); device Power:MFR-25FBF52-3K65 -> rcl:R-US_0207/5V
- R4: value 2k2Ω -> 51.1 kΩ
- R41: value 3.6k -> 1MΩ; device Power:MFR-25FBF52-3K65 -> rcl:R-US_0207/5V
- R42: value 51.1kΩ -> 1KΩ; device Power:MFR-25FBF52-51K1 -> rcl:R-US_0207/5V
- R43: value 3.6k -> 10kΩ; device Power:MFR-25FBF52-3K65 -> rcl:R-US_0207/5V
- R44: value 1MΩ -> 47kΩ
- R5: value 47kΩ -> 373.65 kΩ
- R6: value 47kΩ -> 24.9 kΩ
- R7: value (none) -> 8.06 kΩ; device Power:MFR-25FBF52-3K65 -> rcl:R-US_0207/5V
- R8: value 10kΩ -> 24.9 kΩ
- R9: value 180Ω -> 17.4 kΩ
- U$1: value TEST -> BAT+
- U$2: value TEST -> +24V
- U$3: value CAP -> +3.3V
- U$4: value BAT+ -> CAP
- U$5: value +24V -> TEST
- U$6: value +3.3V -> CAP
- U$7: value CAP -> TEST
- U1: value ATMEGA1284P-PU -> TL431BQLP; device Atmel_By_element14_Batch_1-00:ATMEGA1284P-PU -> Power:TL431BQLP
- U3: value TL431BQLP -> ATMEGA1284P-PU; device Power:TL431BQLP -> Atmel_By_element14_Batch_1-00:ATMEGA1284P-PU
Connections:
- removed net ARMED_SENSE: ARMED.C, PAD2.P, U1.PD6
- removed net N$33: ARMED.A, R9.1
- removed net RELAY_ARM: U1.PC5
- new net EMATCH_SENSE_1: ARMED1.C, R33.1, U3.PD6
- new net EMATCH_SENSE_2: ARMED2.C, R32.1, U3.PD7
- new net N$35: R24.2, T4.B
- new net N$67: C12.1, R13.1
- new net N$75: C10.1, R11.1
- new net N$84: ARMED2.A, R15.2
- new net N$85: ARMED1.A, R12.1
- net +12.0: now also C2.+, C3.1, D1.C, R22.1, R23.1, R25.1, R26.1, R27.1, R28.1, R31.1, R34.1, R35.1, R36.1, R38.1, R39.1, R4.1, R40.1, U$2.P$1; no longer C25.+, D3.C, R15.11, R16.11, R17.11, R18.11, R19.11, R20.11, R21.11, R22.11, R23.11, R24.11, R25.11, R26.11, R27.11, R28.11, R29.11, R42.11
- net 12V_ENABLE: now also R24.1, R29.2, U$5.P$1, U3.PC5; no longer U$2.P$1
- net ACCEL_INT: now also IC5.INT1, U3.PC3; no longer IC2.INT1, U1.PC3
- net ALT_INT: now also IC6.INT1, U3.PC2; no longer IC3.INT1, U1.PC2
- net AREF: now also C32.1, U3.AREF; no longer C14.1, U1.AREF
- net AVCC: now also C31.2, C37.2, L3.2, Q4.VDD, Q5.VDD, U3.AVCC; no longer C11.2, C9.2, L1.2, Q1.VDD, Q2.VDD, U1.AVCC
- net A_GND: now also C31.1, C32.2, C35.2, C37.1, Q4.GND, Q5.GND, R47.1, R48.2, U3.GND; no longer C11.1, C12.2, C14.2, C9.1, Q1.GND, Q2.GND, R2.22, R6.1, U1.GND
- net BAT+: now also Q1.S, R1.1, R2.1, R46.2, U$1.P$1; no longer Q4.S, R33.11, R34.11, R5.2, U$8.P$1
- net BAT_REF: now also C35.1, R46.1, R47.2, U3.PA7; no longer C12.1, R5.1, R6.2, U1.PA7
- net CAP_DISCHARGE: now also R18.1, U3.PD4; no longer R13.11, U1.PD4
- net CAP_REF: now also R45.2, R48.1, U$7.P$1, U3.PA0; no longer R2.11, R7.22, U$1.P$1, U1.PA0
- net DEBUG_LED: now also U3.PB0; no longer U1.PB0
- net EEPROM2_CS: now also IC1.!CS, R30.1, U3.PB1; no longer IC6.!CS, R44.1, U1.PB1
- net EEPROM_CS: now also IC2.!CS, R37.1, U3.PB3; no longer IC5.!CS, R14.1, U1.PB3
- net FB1: now also R4.2, R5.1; no longer R37.11, R42.22
- net GND: now also C1.-, C11.-, C12.2, C14.-, C15.-, C18.2, C2.-, C22.1, C23.2, C24.2, C25.2, C26.2, C27.2, C28.2, C30.-, C34.-, C36.2, C4.-, C6.2, C8.2, C9.2, IC1.!WP, IC1.GND, IC2.!WP, IC3.GND@1, IC3.GND@2, IC3.GND@3, IC3.GND@4, IC4.RSVD1, IC4.RSVD10, IC4.RSVD2, IC4.RSVD3, IC4.RSVD4, IC4.RSVD5, IC4.RSVD6, IC4.RSVD7, IC4.RSVD8, IC4.RSVD9, IC4.SA0/MISO, IC4.VSS1, IC4.VSS2, IC4.VSS3, IC4.VSS4, IC5.GND_2, IC5.GND_3, IC5.SDO/ALT_ADDRESS, R17.1, R19.1, R29.1, R3.2, R32.2, R33.2, R42.2, R5.2, R7.1, R9.1, T4.E, U$4.P$1, U1.ANODE, U3.GND_2, XLR1.GND, XLR1.OUT2; no longer C1.2, C10.2, C15.2, C18.1, C2.2, C22.-, C23.-, C24.-, C25.-, C26.-, C27.-, C30.2, C31.2, C32.2, C4.2, C6.-, C8.-, DC1.GND, IC1.RSVD1, IC1.RSVD10, IC1.RSVD2, IC1.RSVD3, IC1.RSVD4, IC1.RSVD5, IC1.RSVD6, IC1.RSVD7, IC1.RSVD8, IC1.RSVD9, IC1.SA0/MISO, IC1.VSS1, IC1.VSS2, IC1.VSS3, IC1.VSS4, IC2.GND_2, IC2.GND_3, IC2.SDO/ALT_ADDRESS, IC3.GND, IC4.GND@1, IC4.GND@2, IC4.GND@3, IC4.GND@4, IC5.!WP, IC6.!WP, PAD1.P, R10.2, R12.11, R31.22, R35.11, R36.11, R37.22, R39.11, U$3.P$1, U1.GND_2, U3.ANODE
- net GPS_FIX: now also IC3.3D-FIX; no longer IC4.3D-FIX
- net GYRO_INT: now also IC4.INT1, U3.PC4; no longer IC1.INT1, U1.PC4
- net MAIN_TRIGGER: now also R14.1, R16.1, R17.2, U3.PD5; no longer R39.22, R41.11, R43.11, U1.PD5
- net MISO: now also IC1.SO, IC2.SO, U3.PB6; no longer IC5.SO, IC6.SO, U1.PB6
- net MOSI: now also IC1.SI, IC2.SI, U3.PB5; no longer IC5.SI, IC6.SI, U1.PB5
- net N$1: now also C27.1, IC4.VREGD; no longer C5.1, IC1.VREGD
- net N$10: now also C9.1, R8.1; no longer C32.1, R38.11
- net N$11: now also R6.1; no longer R32.11
- net N$12: now also C6.1; no longer C29.1
- net N$13: now also C10.2, L2.1, R13.2; no longer C28.2, L3.1
- net N$15: now also R10.1, R9.2; no longer R35.22, R40.11
- net N$16: now also D3.C, R11.2; no longer C28.1, D1.C
- net N$2: now also IC4.!RST, R44.2; no longer IC1.!RST, R1.2
- net N$3: now also C36.1, IC6.CAP; no longer C13.1, IC3.CAP
- net N$30: now also Q2.S, R21.1, R22.2, R23.2, R25.2, R26.2, R27.2, R28.2, R31.2, R34.2, R35.2, R36.2, R38.2, R39.2, R40.2; no longer DC1.SW, XLR1.GND, XLR1.OUT2
- net N$31: now also Q2.G, R21.2, T4.C; no longer PAD4.P, XLR2.OUT2, XLR2.OUT4
- net N$34: now also R20.2, T3.C; no longer R30.11, T1.C
- net N$4: now also IC3.EX_ANT; no longer IC4.EX_ANT
- net N$5: now also C8.1; no longer C31.1
- net N$6: now also R7.2; no longer R36.22
- net N$69: now also Q1.G, R1.2, U1.CATHODE; no longer Q4.G, R33.22, U3.CATHODE
- net N$7: now also R8.2; no longer R38.22
- net N$70: now also R2.2, R3.1, U1.REF; no longer R31.11, R34.22, U3.REF
- net N$71: now also R42.1; no longer R10.1
- net N$77: now also PAD3.P, R15.1, T1.C, XLR2.OUT5; no longer T3.C, XLR2.OUT3
- net N$78: now also PAD2.P, R12.2, XLR2.OUT4; no longer XLR2.OUT5
- net N$79: now also R16.2, T2.B; no longer R43.22, T3.B
- net N$8: now also D1.A, L1.2; no longer D3.A, L2.2, U$5.P$1
- net N$80: now also R14.2, T1.B; no longer R41.22, T2.B
- net N$81: now also C11.+, C15.+, C4.+, PAD1.P, Q2.D, R20.1, R45.1, U$6.P$1, XLR2.OUT2, XLR2.OUT3; no longer C22.+, C23.+, C24.+, PAD3.P, R15.22, R16.22, R17.22, R18.22, R19.22, R20.22, R21.22, R22.22, R23.22, R24.22, R25.22, R26.22, R27.22, R28.22, R29.22, R30.22, R7.11, U$7.P$1
- net N$82: now also R18.2, R19.2, T3.B; no longer R12.22, R13.22, T1.B
- net N$9: now also C5.1, R6.2; no longer C30.1, R32.22
- net PWR_JUNC: now also C1.+, C7.1, L1.1, Q1.D; no longer C27.+, DC1.+12V, L2.1, Q4.D, U$4.P$1
- net RADIO_CS: now also R41.1, U3.PB4; no longer R11.1, U1.PB4
- net RADIO_INT: now also U3.PB2; no longer U1.PB2
- net RESET: now also R43.1, U3.~RESET; no longer R8.1, U1.~RESET
- net RXD0: now also U3.PD0; no longer U1.PD0
- net RXD1: now also IC3.TX, U3.PD2; no longer IC4.TX, U1.PD2
- net SCK: now also IC1.SCK, IC2.SCK, U3.PB7; no longer IC5.SCK, IC6.SCK, U1.PB7
- net SCL: now also IC4.SCL/SCLK, IC5.SCL/SCLK, IC6.SCL, R49.1, U3.PC0; no longer IC1.SCL/SCLK, IC2.SCL/SCLK, IC3.SCL, R3.1, U1.PC0
- net SDA: now also IC4.SDA/MOSI, IC5.SDA/SDI/SDIO, IC6.SDA, R50.1, U3.PC1; no longer IC1.SDA/MOSI, IC2.SDA/SDI/SDIO, IC3.SDA, R4.1, U1.PC1
- net TEMP: now also Q5.VOUT, U3.PA1; no longer Q1.VOUT, U1.PA1
- net TEMP2: now also Q4.VOUT, U3.PA2; no longer Q2.VOUT, U1.PA2
- net TXD0: now also U3.PD1; no longer U1.PD1
- net TXD1: now also IC3.RX, U3.PD3; no longer IC4.RX, U1.PD3
- net VCC: now also C13.1, C14.+, C17.1, C19.1, D3.A, IC1.!HOLD, IC1.VCC, IC2.!HOLD, IC2.VCC, L2.2, R10.2, R30.2, R37.2, SJ200.1, U$3.P$1; no longer C21.1, C26.+, C33.1, D1.A, IC5.!HOLD, IC5.VCC, IC6.!HOLD, IC6.VCC, L3.2, R14.2, R40.22, R44.2, R9.2, SJ6.1, U$6.P$1
- net VCC_ACCEL: now also C28.1, C29.1, C30.+, IC5.!CS, IC5.VDD_I/O, IC5.VS, SJ4.2; no longer C4.1, C6.+, C7.1, IC2.!CS, IC2.VDD_I/O, IC2.VS, SJ3.2
- net VCC_ALT: now also C33.1, C34.+, IC6.VDD, IC6.VDDIO, SJ5.2; no longer C10.1, C8.+, IC3.VDD, IC3.VDDIO, SJ2.2
- net VCC_GPS: now also C22.2, IC3.VCC, SJ2.2; no longer C18.2, IC4.VCC, SJ5.2
- net VCC_GYRO: now also C23.1, C25.1, C26.1, IC4.I2C/!SPI, IC4.VDDIO, IC4.VDD_33, R44.1, SJ3.2; no longer C1.1, C2.1, C3.1, IC1.I2C/!SPI, IC1.VDDIO, IC1.VDD_33, R1.1, SJ1.2
- net VCC_MCU: now also C24.1, L3.1, R41.2, R43.2, R49.2, R50.2, SJ1.2, U3.VCC; no longer C15.1, L1.1, R11.2, R3.2, R4.2, R8.2, SJ6.2, U1.VCC
- net VCC_XB: now also C16.1, C18.1, SJ200.2; no longer C19.1, C20.1, SJ4.2
- net XTAL1: now also C20.1, U3.XTAL1; no longer C17.1, U1.XTAL1
- net XTAL2: now also C21.1, U3.XTAL2; no longer C16.1, U1.XTAL2
